File: kicad/ACS712_AmMeter/ACS712_AmMeter/ACS712_AmMeter.kicad_pcb (KiCad board)
At the start: 2 copper layers, 94 x 71.1 mm, 37 parts, among them J1 BATT_IN, J2 GND, J3 I2C_PIN, J4 POS_IN, J5 NEG_IN, U1 NJM2396, U2 TLE2426xLP, U3 OLED_SSD1306_I2C, U4 NJU7032D

Commit message: Add: logo bule, Update: KiCad design
Parts:
- moved R5 28.4 mm to (132.1, 78.7), turned to 180 degrees
- moved R4 25.9 mm to (129.5, 81.3), turned to 180 degrees
- moved J3 18.3 mm to (109.2, 83.8), turned to 0 degrees
- moved R1 7.62 mm to (152.4, 66.0), turned to 270 degrees
- moved C4 7.18 mm to (167.6, 88.9)
- moved A1 6.35 mm to (119.4, 101.6)
- moved C5 5.68 mm to (152.4, 88.9)
- moved R2 5.68 mm to (149.9, 73.7), turned to 90 degrees
- moved C8 5.08 mm to (154.9, 111.8)
- moved C9 5.08 mm to (172.6, 114.3)
- moved C6 5.08 mm to (149.9, 101.6)
- moved U4 5.08 mm to (157.5, 101.6)
- moved C10 5.08 mm to (162.6, 99.1)
- moved C11 5.08 mm to (160.0, 111.8)
- moved C7 5.08 mm to (172.7, 104.1)
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Routing:
- net GND: track 0.00 -> 212.2 mm
- net +5V: track 0.00 -> 148.6 mm, vias 0 -> 6
- net +2V5: track 0.00 -> 96.2 mm, vias 0 -> 2
- net +BATT: track 0.00 -> 58.7 mm, vias 0 -> 2
- net V_NEG: track 0.00 -> 39.2 mm, vias 0 -> 2
- net V_POS: track 0.00 -> 18.8 mm
- net Net-(J4-Pad2): track 0.00 -> 12.7 mm, vias 0 -> 2
- net Net-(J5-Pad2): track 0.00 -> 11.2 mm
- net Net-(C9-Pad1): track 0.00 -> 9.80 mm
- net Net-(C6-Pad1): track 0.00 -> 8.67 mm
- net Net-(C7-Pad1): track 0.00 -> 8.67 mm
- net Net-(C8-Pad1): track 0.00 -> 7.62 mm
- net Net-(D1-Pad2): track 0.00 -> 5.08 mm
- net V_BATT: track 0.00 -> 2.54 mm

Commit message: Update: Board design
Parts:
- added G***: LOGO, myfootprint:Silk_PNPN_Manufactory_600dpi, F.Cu at (139.7, 124.5)
- added J6: CONFIG_SW, Connector_PinHeader_2.54mm:PinHeader_1x02_P2.54mm_Vertical, F.Cu at (142.2, 86.4)
- A1: value Arduino_PRO-MINI-2 -> Arduino_PRO-MINI-2-ArduinoProMini-simple; footprint ArduinoProMini:PRO-MINI-2 -> myfootprint:Arduino-PRO-MINI-2-simple
- R4, R5: value 4.7k -> 2.2k
- U1: footprint Package_TO_SOT_THT:TO-220-4_Vertical -> myfootprint:NJM2396_Vertical
- moved C2 49.3 mm to (116.8, 78.7), turned to 180 degrees
- moved BZ1 49.3 mm to (134.6, 81.3), turned to 90 degrees
- moved R5 38.1 mm to (132.1, 116.8), turned to 0 degrees
- moved J3 35.9 mm to (134.6, 109.2), turned to 180 degrees
- moved R4 33.1 mm to (132.1, 114.3), turned to 0 degrees
- moved U3 21.7 mm to (118.1, 106.7), turned to 0 degrees
- moved A1 9.25 mm to (121.9, 92.7), turned to 90 degrees
Connections:
- A1 pad A0: V_POS -> V_NEG
- A1 pad A1: V_NEG -> V_POS
- A1 pad D11: (no net) -> Net-(A1-PadD11)
- BZ1 pad 1: Net-(A1-PadD10) -> Net-(A1-PadD11)
Routing:
- net +5V: track 148.6 -> 276.3 mm, vias 6 -> 10
- net GND: track 212.2 -> 336.0 mm, vias 0 -> 2
- net V_NEG: track 39.2 -> 87.4 mm
- net /SCL: track 0.00 -> 46.5 mm
- net /SDA: track 0.00 -> 41.8 mm
- net V_BATT: track 2.54 -> 41.7 mm, vias 0 -> 2
- net V_POS: track 18.8 -> 47.4 mm
- net Net-(A1-PadD10): track 0.00 -> 5.08 mm
- net Net-(A1-PadD11): track 0.00 -> 5.08 mm

Commit message: Update: Board design
Parts:
- removed G***: LOGO, myfootprint:Silk_PNPN_Manufactory_600dpi
- A1: value Arduino_PRO-MINI-2-ArduinoProMini-simple -> Arduino_PRO-MINI
- J6: value CONFIG_SW -> CAL_SW

Commit message: Ubdate: Board design
Parts:
- added G***: LOGO, myfootprint:Silk_PNPN_Manufactory_600dpi, F.Cu at (139.1, 125.7)
- added J7: +5V_OUT, Connector_PinHeader_2.54mm:PinHeader_1x02_P2.54mm_Vertical, F.Cu at (188.0, 94.0)
- J1: footprint Connector_PinHeader_2.54mm:PinHeader_1x02_P2.54mm_Vertical -> Connector_JST:JST_XH_B2B-XH-A_1x02_P2.50mm_Vertical
- J2: value GND -> TP_GND
- turned J1 to 270 degrees
Routing:
- net +5V: track 276.3 -> 301.8 mm
- net GND: track 336.0 -> 338.5 mm

Commit message: Soldering completed
Parts:
- moved J6 40.7 mm to (101.6, 88.9)
- moved G*** 1.42 mm to (139.7, 124.5)
Connections:
- A1 pad D10: Net-(A1-PadD10) -> (no net)
- A1 pad D2: (no net) -> Net-(A1-PadD2)
- J6 pad 1: Net-(A1-PadD10) -> Net-(A1-PadD2)
Routing:
- net Net-(A1-PadD2): track 0.00 -> 30.5 mm, vias 0 -> 2
- net GND: track 338.5 -> 329.5 mm, vias 2 -> 0
- net Net-(A1-PadD10): track 5.08 -> 0.00 mm
