File: kicad/ACS712_AmMeter/ACS712_AmMeter/ACS712_AmMeter.sch (KiCad schematic (older format))
At the start: 37 parts, among them J1 BATT_IN, J2 GND, J3 I2C_PIN, J4 POS_IN, J5 NEG_IN, U1 NJM2396, U2 TLE2426xLP, U3 OLED_SSD1306_I2C, U4 NJU7032D

Commit message: Update: Board design
Parts:
- removed A1: Arduino_PRO-MINI-2, ArduinoProMini:PRO-MINI-2, symbol ACS712_AmMeter-rescue:Arduino_PRO-MINI-2-ArduinoProMini-eagle-import
- added A1: Arduino_PRO-MINI-2-ArduinoProMini-simple, myfootprint:Arduino-PRO-MINI-2-simple, symbol mylib:Arduino_PRO-MINI-2-ArduinoProMini-simple
- added J6: CONFIG_SW, Connector_PinHeader_2.54mm:PinHeader_1x02_P2.54mm_Vertical, symbol Connector_Generic:Conn_01x02
- R4, R5: value 4.7k -> 2.2k
- U1: footprint Package_TO_SOT_THT:TO-220-4_Horizontal_TabDown -> myfootprint:NJM2396_Vertical
Connections:
- net +5V: now also A1.VCC
- net GND: now also A1.GND, J6.2 (Pin_2)
- net SCL: now also A1.A5
- net SDA: now also A1.A4
- net V_BATT: now also A1.A2
- net V_NEG: now also A1.A0
- net V_POS: now also A1.A1
- net at BZ1.1 (-): now also A1.D11
- new net: A1.D10, J6.1 (Pin_1)
- no-connect marks 26 -> 19
Other:
- moved on the sheet: BZ1
Changed lines of the file:
@@
 EESchema Schematic File Version 4
 LIBS:ACS712_AmMeter-cache
-LIBS:ACS712_AmMeter_Analog-cache
 EELAYER 30 0
 EELAYER END
@@
 Sheet 1 1
 Title "ACS712_AmMeter_Digital_Board"
-Date "2020-01-19"
-Rev "Ver. 0.91"
+Date "2020-01-25"
+Rev "Ver. 0.92"
 Comp "PNPN Manufactory"
 Comment1 ""
@@
 Wire Wire Line
 	2700 5450 2900 5450
-Wire Wire Line
-	2700 5350 2900 5350
-NoConn ~ 2800 4550
-NoConn ~ 2700 4550
-NoConn ~ 2600 4550
-NoConn ~ 2500 4550
-NoConn ~ 2400 4550
-NoConn ~ 2300 4550
 NoConn ~ 1700 5050
 NoConn ~ 1700 5150
@@
 NoConn ~ 1700 5950
 NoConn ~ 1700 6150
-NoConn ~ 3400 6050
 NoConn ~ 3400 5950
 NoConn ~ 3400 5850
@@
 NoConn ~ 2700 5650
 NoConn ~ 2700 5750
-$Comp
-L ACS712_AmMeter-rescue:Arduino_PRO-MINI-2-ArduinoProMini-eagle-import A1
-U 1 1 5E1A783C
-P 2600 5550
-F 0 "A1" H 1950 6400 50  0000 C CNN
-F 1 "Arduino_PRO-MINI-2" H 2300 4700 50  0000 C CNN
-F 2 "ArduinoProMini:PRO-MINI-2" H 2600 5550 50  0001 C CNN
-F 3 "" H 2600 5550 50  0001 C CNN
-	1    2600 5550
-	1    0    0    -1
-$EndComp
 $Comp
 L mylib:OLED_SSD1306_I2C U3
@@
 P 5400 5150
 F 0 "R4" H 5470 5196 50  0000 L CNN
-F 1 "4.7k" H 5470 5105 50  0000 L CNN
+F 1 "2.2k" H 5470 5105 50  0000 L CNN
 F 2 "Resistor_THT:R_Axial_DIN0207_L6.3mm_D2.5mm_P7.62mm_Horizontal" V 5330 5150 50  0001 C CNN
 F 3 "~" H 5400 5150 50  0001 C CNN
@@
 P 5700 5150
 F 0 "R5" H 5770 5196 50  0000 L CNN
-F 1 "4.7k" H 5770 5105 50  0000 L CNN
+F 1 "2.2k" H 5770 5105 50  0000 L CNN
 F 2 "Resistor_THT:R_Axial_DIN0207_L6.3mm_D2.5mm_P7.62mm_Horizontal" V 5630 5150 50  0001 C CNN
 F 3 "~" H 5700 5150 50  0001 C CNN
@@
 L Device:Buzzer BZ1
 U 1 1 5E3F79F4
-P 3800 6250
-F 0 "BZ1" H 3805 6540 50  0000 C CNN
-F 1 "Buzzer" H 3805 6449 50  0000 C CNN
-F 2 "Buzzer_Beeper:Buzzer_12x9.5RM7.6" V 3775 6350 50  0001 C CNN
-F 3 "~" V 3775 6350 50  0001 C CNN
-	1    3800 6250
+P 4050 6150
+F 0 "BZ1" H 4055 6440 50  0000 C CNN
+F 1 "Buzzer" H 4055 6349 50  0000 C CNN
+F 2 "Buzzer_Beeper:Buzzer_12x9.5RM7.6" V 4025 6250 50  0001 C CNN
+F 3 "~" V 4025 6250 50  0001 C CNN
+	1    4050 6150
 	1    0    0    -1
 $EndComp
@@
 	5150 5500 5150 5600
 NoConn ~ 1700 6050
-Wire Wire Line
-	3400 6150 3700 6150
-Wire Wire Line
-	3700 6350 3500 6350
-Connection ~ 3500 6350
-Wire Wire Line
-	3500 6350 3500 6500
 $Comp
 L Device:D_Schottky D2
@@
 F 0 "U1" H 4000 3065 50  0000 C CNN
 F 1 "NJM2396" H 4000 2974 50  0000 C CNN
-F 2 "Package_TO_SOT_THT:TO-220-4_Horizontal_TabDown" H 4000 3050 50  0001 C CNN
+F 2 "myfootprint:NJM2396_Vertical" H 4000 3050 50  0001 C CNN
 F 3 "https://www.njr.co.jp/products/semicon/PDF/old_pdf/NJM2396_J.pdf" H 4000 2800 50  0001 C CNN
 	1    4000 2800
@@
 	3850 5450 3500 5450
 Connection ~ 3500 5450
-Wire Wire Line
-	3500 5450 3500 6350
 Text GLabel 4000 5550 2    50   Input ~ 0
 V_BATT
+Text GLabel 4000 5750 2    50   Input ~ 0
+V_NEG
 Text GLabel 4000 5650 2    50   Input ~ 0
-V_NEG
-Text GLabel 4000 5750 2    50   Input ~ 0
 V_POS
 $Comp
@@
 L power:GNDD #PWR08
 U 1 1 5E377BD9
-P 3500 6500
-F 0 "#PWR08" H 3500 6250 50  0001 C CNN
-F 1 "GNDD" H 3504 6345 50  0000 C CNN
-F 2 "" H 3500 6500 50  0001 C CNN
-F 3 "" H 3500 6500 50  0001 C CNN
-	1    3500 6500
+P 3500 6850
+F 0 "#PWR08" H 3500 6600 50  0001 C CNN
+F 1 "GNDD" H 3504 6695 50  0000 C CNN
+F 2 "" H 3500 6850 50  0001 C CNN
+F 3 "" H 3500 6850 50  0001 C CNN
+	1    3500 6850
 	1    0    0    -1
 $EndComp
@@
 Wire Wire Line
 	7500 3100 7550 3100
+$Comp
+L mylib:Arduino_PRO-MINI-2-ArduinoProMini-simple A1
+U 1 1 5E28BA03
+P 2600 5550
+F 0 "A1" H 2550 6515 50  0000 C CNN
+F 1 "Arduino_PRO-MINI-2-ArduinoProMini-simple" H 2550 6424 50  0000 C CNN
+F 2 "myfootprint:Arduino-PRO-MINI-2-simple" H 2600 5550 50  0001 C CNN
+F 3 "" H 2600 5550 50  0001 C CNN
+	1    2600 5550
+	1    0    0    -1
+$EndComp
+Wire Wire Line
+	2700 5350 2900 5350
+Wire Wire Line
+	3400 6050 3950 6050
+$Comp
+L Connector_Generic:Conn_01x02 J6
+U 1 1 5E2C9B1F
+P 4100 6550
+F 0 "J6" H 4018 6767 50  0000 C CNN
+F 1 "CONFIG_SW" H 4018 6676 50  0000 C CNN
+F 2 "Connector_PinHeader_2.54mm:PinHeader_1x02_P2.54mm_Vertical" H 4100 6550 50  0001 C CNN
+F 3 "~" H 4100 6550 50  0001 C CNN
+	1    4100 6550
+	1    0    0    -1
+$EndComp
+Wire Wire Line
+	3800 6150 3800 6550
+Wire Wire Line
+	3800 6550 3900 6550
+Wire Wire Line
+	3400 6150 3800 6150
+Wire Wire Line
+	3900 6650 3500 6650
+Connection ~ 3500 6650
+Wire Wire Line
+	3500 6650 3500 6850
+Wire Wire Line
+	3500 5450 3500 6250
+Wire Wire Line
+	3950 6250 3500 6250
+Connection ~ 3500 6250
+Wire Wire Line
+	3500 6250 3500 6650
 $EndSCHEMATC

Commit message: Update: Board design
Parts:
- A1: value Arduino_PRO-MINI-2-ArduinoProMini-simple -> Arduino_PRO-MINI
- J6: value CONFIG_SW -> CAL_SW
Changed lines of the file:
@@
 P 2600 5550
 F 0 "A1" H 2550 6515 50  0000 C CNN
-F 1 "Arduino_PRO-MINI-2-ArduinoProMini-simple" H 2550 6424 50  0000 C CNN
+F 1 "Arduino_PRO-MINI" H 2550 6424 50  0000 C CNN
 F 2 "myfootprint:Arduino-PRO-MINI-2-simple" H 2600 5550 50  0001 C CNN
 F 3 "" H 2600 5550 50  0001 C CNN
@@
 P 4100 6550
 F 0 "J6" H 4018 6767 50  0000 C CNN
-F 1 "CONFIG_SW" H 4018 6676 50  0000 C CNN
+F 1 "CAL_SW" H 4018 6676 50  0000 C CNN
 F 2 "Connector_PinHeader_2.54mm:PinHeader_1x02_P2.54mm_Vertical" H 4100 6550 50  0001 C CNN
 F 3 "~" H 4100 6550 50  0001 C CNN

Commit message: Ubdate: Board design
Parts:
- added J7: +5V_OUT, Connector_PinHeader_2.54mm:PinHeader_1x02_P2.54mm_Vertical, symbol Connector_Generic:Conn_01x02
- J1: footprint Connector_PinHeader_2.54mm:PinHeader_1x02_P2.54mm_Vertical -> Connector_JST:JST_XH_B2B-XH-A_1x02_P2.50mm_Vertical
- J2: value GND -> TP_GND
Connections:
- net +5V: now also J7.1 (Pin_1)
- net GND: now also J7.2 (Pin_2)
Other:
- moved on the sheet: H1, H2, H3, H4
Changed lines of the file:
@@
 Sheet 1 1
 Title "ACS712_AmMeter_Digital_Board"
-Date "2020-01-25"
-Rev "Ver. 0.92"
+Date "2020-01-27"
+Rev "Ver. 0.93"
 Comp "PNPN Manufactory"
 Comment1 ""
@@
 L Mechanical:MountingHole H1
 U 1 1 5E40C003
-P 3400 1250
-F 0 "H1" H 3500 1296 50  0000 L CNN
-F 1 "MountingHole" H 3500 1205 50  0000 L CNN
-F 2 "MountingHole:MountingHole_3.2mm_M3" H 3400 1250 50  0001 C CNN
-F 3 "~" H 3400 1250 50  0001 C CNN
-	1    3400 1250
+P 4300 1250
+F 0 "H1" H 4400 1296 50  0000 L CNN
+F 1 "MountingHole" H 4400 1205 50  0000 L CNN
+F 2 "MountingHole:MountingHole_3.2mm_M3" H 4300 1250 50  0001 C CNN
+F 3 "~" H 4300 1250 50  0001 C CNN
+	1    4300 1250
 	1    0    0    -1
 $EndComp
@@
 L Mechanical:MountingHole H2
 U 1 1 5E40C738
-P 3400 1500
-F 0 "H2" H 3500 1546 50  0000 L CNN
-F 1 "MountingHole" H 3500 1455 50  0000 L CNN
-F 2 "MountingHole:MountingHole_3.2mm_M3" H 3400 1500 50  0001 C CNN
-F 3 "~" H 3400 1500 50  0001 C CNN
-	1    3400 1500
+P 4300 1500
+F 0 "H2" H 4400 1546 50  0000 L CNN
+F 1 "MountingHole" H 4400 1455 50  0000 L CNN
+F 2 "MountingHole:MountingHole_3.2mm_M3" H 4300 1500 50  0001 C CNN
+F 3 "~" H 4300 1500 50  0001 C CNN
+	1    4300 1500
 	1    0    0    -1
 $EndComp
@@
 L Mechanical:MountingHole H3
 U 1 1 5E40CD16
-P 4150 1250
-F 0 "H3" H 4250 1296 50  0000 L CNN
-F 1 "MountingHole" H 4250 1205 50  0000 L CNN
-F 2 "MountingHole:MountingHole_3.2mm_M3" H 4150 1250 50  0001 C CNN
-F 3 "~" H 4150 1250 50  0001 C CNN
-	1    4150 1250
+P 5050 1250
+F 0 "H3" H 5150 1296 50  0000 L CNN
+F 1 "MountingHole" H 5150 1205 50  0000 L CNN
+F 2 "MountingHole:MountingHole_3.2mm_M3" H 5050 1250 50  0001 C CNN
+F 3 "~" H 5050 1250 50  0001 C CNN
+	1    5050 1250
 	1    0    0    -1
 $EndComp
@@
 L Mechanical:MountingHole H4
 U 1 1 5E40D241
-P 4150 1500
-F 0 "H4" H 4250 1546 50  0000 L CNN
-F 1 "MountingHole" H 4250 1455 50  0000 L CNN
-F 2 "MountingHole:MountingHole_3.2mm_M3" H 4150 1500 50  0001 C CNN
-F 3 "~" H 4150 1500 50  0001 C CNN
-	1    4150 1500
+P 5050 1500
+F 0 "H4" H 5150 1546 50  0000 L CNN
+F 1 "MountingHole" H 5150 1455 50  0000 L CNN
+F 2 "MountingHole:MountingHole_3.2mm_M3" H 5050 1500 50  0001 C CNN
+F 3 "~" H 5050 1500 50  0001 C CNN
+	1    5050 1500
 	1    0    0    -1
 $EndComp
@@
 F 0 "J1" H 1668 3017 50  0000 C CNN
 F 1 "BATT_IN" H 1668 2926 50  0000 C CNN
-F 2 "Connector_PinHeader_2.54mm:PinHeader_1x02_P2.54mm_Vertical" H 1750 2800 50  0001 C CNN
+F 2 "Connector_JST:JST_XH_B2B-XH-A_1x02_P2.50mm_Vertical" H 1750 2800 50  0001 C CNN
 F 3 "~" H 1750 2800 50  0001 C CNN
 	1    1750 2800
@@
 P 2750 1300
 F 0 "J2" H 2668 1517 50  0000 C CNN
-F 1 "GND" H 2668 1426 50  0000 C CNN
+F 1 "TP_GND" H 2668 1426 50  0000 C CNN
 F 2 "Connector_PinHeader_2.54mm:PinHeader_1x02_P2.54mm_Vertical" H 2750 1300 50  0001 C CNN
 F 3 "~" H 2750 1300 50  0001 C CNN
@@
 Wire Wire Line
 	3500 6250 3500 6650
+$Comp
+L Connector_Generic:Conn_01x02 J7
+U 1 1 5E2EB662
+P 3350 1300
+F 0 "J7" H 3268 1517 50  0000 C CNN
+F 1 "+5V_OUT" H 3268 1426 50  0000 C CNN
+F 2 "Connector_PinHeader_2.54mm:PinHeader_1x02_P2.54mm_Vertical" H 3350 1300 50  0001 C CNN
+F 3 "~" H 3350 1300 50  0001 C CNN
+	1    3350 1300
+	-1   0    0    -1
+$EndComp
+$Comp
+L power:GND #PWR032
+U 1 1 5E2EB66C
+P 3700 1450
+F 0 "#PWR032" H 3700 1200 50  0001 C CNN
+F 1 "GND" H 3705 1277 50  0000 C CNN
+F 2 "" H 3700 1450 50  0001 C CNN
+F 3 "" H 3700 1450 50  0001 C CNN
+	1    3700 1450
+	1    0    0    -1
+$EndComp
+$Comp
+L power:+5V #PWR031
+U 1 1 5E2F205B
+P 3700 1200
+F 0 "#PWR031" H 3700 1050 50  0001 C CNN
+F 1 "+5V" H 3715 1373 50  0000 C CNN
+F 2 "" H 3700 1200 50  0001 C CNN
+F 3 "" H 3700 1200 50  0001 C CNN
+	1    3700 1200
+	1    0    0    -1
+$EndComp
+Wire Wire Line
+	3550 1300 3700 1300
+Wire Wire Line
+	3700 1300 3700 1200
+Wire Wire Line
+	3550 1400 3700 1400
+Wire Wire Line
+	3700 1400 3700 1450
 $EndSCHEMATC

Commit message: Soldering completed
Connections:
- net at A1.D10: no longer J6.1 (Pin_1)
- net at A1.D2: now also J6.1 (Pin_1)
Other:
- moved on the sheet: J6
Changed lines of the file:
@@
 Sheet 1 1
 Title "ACS712_AmMeter_Digital_Board"
-Date "2020-01-27"
-Rev "Ver. 0.93"
+Date "2020-01-29"
+Rev "Ver. 0.94"
 Comp "PNPN Manufactory"
 Comment1 ""
@@
 NoConn ~ 1700 5250
 NoConn ~ 1700 5350
-NoConn ~ 1700 5450
 NoConn ~ 1700 5550
 NoConn ~ 1700 5650
@@
 L power:GNDD #PWR08
 U 1 1 5E377BD9
-P 3500 6850
-F 0 "#PWR08" H 3500 6600 50  0001 C CNN
-F 1 "GNDD" H 3504 6695 50  0000 C CNN
-F 2 "" H 3500 6850 50  0001 C CNN
-F 3 "" H 3500 6850 50  0001 C CNN
-	1    3500 6850
+P 3500 6400
+F 0 "#PWR08" H 3500 6150 50  0001 C CNN
+F 1 "GNDD" H 3504 6245 50  0000 C CNN
+F 2 "" H 3500 6400 50  0001 C CNN
+F 3 "" H 3500 6400 50  0001 C CNN
+	1    3500 6400
 	1    0    0    -1
 $EndComp
@@
 L Connector_Generic:Conn_01x02 J6
 U 1 1 5E2C9B1F
-P 4100 6550
-F 0 "J6" H 4018 6767 50  0000 C CNN
-F 1 "CAL_SW" H 4018 6676 50  0000 C CNN
-F 2 "Connector_PinHeader_2.54mm:PinHeader_1x02_P2.54mm_Vertical" H 4100 6550 50  0001 C CNN
-F 3 "~" H 4100 6550 50  0001 C CNN
-	1    4100 6550
-	1    0    0    -1
-$EndComp
-Wire Wire Line
-	3800 6150 3800 6550
-Wire Wire Line
-	3800 6550 3900 6550
-Wire Wire Line
-	3400 6150 3800 6150
-Wire Wire Line
-	3900 6650 3500 6650
-Connection ~ 3500 6650
-Wire Wire Line
-	3500 6650 3500 6850
+P 1300 5450
+F 0 "J6" H 1218 5667 50  0000 C CNN
+F 1 "CAL_SW" H 1218 5576 50  0000 C CNN
+F 2 "Connector_PinHeader_2.54mm:PinHeader_1x02_P2.54mm_Vertical" H 1300 5450 50  0001 C CNN
+F 3 "~" H 1300 5450 50  0001 C CNN
+	1    1300 5450
+	-1   0    0    -1
+$EndComp
 Wire Wire Line
 	3500 5450 3500 6250
@@
 	3950 6250 3500 6250
 Connection ~ 3500 6250
-Wire Wire Line
-	3500 6250 3500 6650
 $Comp
 L Connector_Generic:Conn_01x02 J7
@@
 Wire Wire Line
 	3700 1400 3700 1450
+Wire Wire Line
+	3500 6250 3500 6400
+$Comp
+L power:GNDD #PWR033
+U 1 1 5E32520B
+P 1550 6400
+F 0 "#PWR033" H 1550 6150 50  0001 C CNN
+F 1 "GNDD" H 1554 6245 50  0000 C CNN
+F 2 "" H 1550 6400 50  0001 C CNN
+F 3 "" H 1550 6400 50  0001 C CNN
+	1    1550 6400
+	1    0    0    -1
+$EndComp
+NoConn ~ 3400 6150
+Wire Wire Line
+	1500 5450 1700 5450
+Wire Wire Line
+	1500 5550 1550 5550
+Wire Wire Line
+	1550 5550 1550 6400
 $EndSCHEMATC
